File: EDA files/EEZ DIB AFE3 r1B3.brd (EAGLE design)
At the start: 129 x 68.5 mm, 149 parts, among them IC1 AMC3330QDWERQ1, IC11 ADS131E04IPAGR, IC12 TPS71725DCKR, IC13 TPS72325DBVR, IC2 ULN2803ADWR, IC3 AMC3301DWER, IC4 MCP6004T-I/ST, IC5 DG212BDY-T1-E3, IC6 MCP6001T-I/OT, IC7 DG212BDY-T1-E3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

Commit message: New Rsense values, PCB layout adjustment for mid range Rsense
Parts:
- R13: value 15R -> 10R
- R15: value 50R 0.1% -> 33R 0.1%
- R32: value 0R33 -> GMR100HTBFIR022; device rcl:R1210 -> EEZ_Lib1:R_2512-4WIRE
- R8: value 0R220 -> GMR100HTBFIR022; device rcl:R1210 -> EEZ_Lib1:R_2512-4WIRE
- moved R32 6.99 mm to (85.5, 45.3), turned to 180 degrees
- moved C20 6.82 mm to (118.9, 59.8)
- moved ISEL10A_2 6.82 mm to (114.8, 58.4)
- moved Q3 4.66 mm to (92.4, 38.9), turned to 0 degrees
- moved TVS1 3.96 mm to (80.4, 44.6), turned to 270 degrees
- moved JP6 3.96 mm to (94.4, 45.0)
- moved R35 3.66 mm to (85.5, 49.5)
- moved D4 3.46 mm to (102.8, 45.6)
- moved D5 3.46 mm to (99.5, 45.6)
- moved R31 3.45 mm to (96.6, 45.0)
- moved R30 3.24 mm to (88.2, 41.8), turned to 0 degrees
- moved Q4 2.12 mm to (89.1, 38.9), turned to 0 degrees
- moved D8 1.27 mm to (102.8, 38.8)
- moved D9 1.27 mm to (99.5, 38.8)
- moved D6 1.27 mm to (99.5, 32.0)
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Connections:
- net N$18 renamed HI_SENSE+
- removed net N$141: F5.2, ISEL10A_2.14, ISEL10A_2.24
- removed net N$71: F2.2, ISEL10A_1.24, R8.2
- new net HI_FORCE+: ISEL10A_1.12, R11.2, R8.1, R8.1S
- new net LOW_SENSE+: ISEL10A_1.24, R8.2S
- new net LO_FORCE-: F2.2, R8.2
- new net N$27: IC7.10, R32.2S
- net AIN4P: now also F5.2
- net HI_CURR#1: no longer R32.1, R35.2S
- net ISEL#3: now also X3.15
- net N$170: no longer IC7.10
- net N$19: now also R32.1, R32.1S, R35.2S; no longer ISEL10A_1.12, R11.2, R8.1
Routing:
- net ISEL#3: track 19.0 -> 77.2 mm, vias 3 -> 5
- net HI_CURR#1: track 7.50 -> 41.0 mm, vias 0 -> 4
- net HI_FORCE+: track 0.00 -> 31.8 mm, vias 0 -> 14
- net N$19: track 33.1 -> 7.37 mm
- net N$71: track 21.6 -> 0.00 mm, vias 4 -> 0
- net N$141: track 17.8 -> 0.00 mm
- net N$27: track 0.00 -> 14.6 mm, vias 0 -> 2
- net LO_FORCE-: track 0.00 -> 14.1 mm, vias 0 -> 4
- net N$182: track 73.2 -> 61.7 mm
- net LOW_SENSE+: track 0.00 -> 10.5 mm
- net AIN4P: track 70.3 -> 79.6 mm, vias 0 -> 6
- net AIN4P_FUSED: track 29.9 -> 22.2 mm, vias 0 -> 2
- net N$170: track 19.2 -> 11.9 mm
- net N$30: track 20.3 -> 26.4 mm
- net ISEL10A_R4_OUT: track 73.6 -> 78.9 mm, vias 2 -> 3
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- added copper zone on layer 16, net AIN2N
- added copper zone on layer 1, net AIN4N
- added copper zone on layer 1, net AIN4P
- added copper zone on layer 16, net HI_CURR#1
- added copper zone on layer 1, net HI_FORCE+
- added copper zone on layer 16, net HI_FORCE+
- added copper zone on layer 1, net LO_FORCE-
- removed copper zone on layer 1, net HI_CURR#1
- removed copper zone on layer 1, net N$19
- removed copper zone on layer 1, net N$71
Other:
- outline, holes or cut-outs redrawn
- board text added: "EEZ DIB AFE3 (05/2021 r1B3)"
- board text removed: "EEZ DIB AFE3 (04/2021 r1B2)"

Commit message: R30 value corrected
Parts:
- R30: value 33R -> 20R
Changed lines of the file:
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@@
 <layer number="131" name="tAdjust" color="7" fill="1" visible="no" active="no"/>
 <layer number="132" name="bAdjust" color="7" fill="1" visible="no" active="no"/>
-<layer number="133" name="DNP_top" color="12" fill="1" visible="no" active="yes"/>
+<layer number="133" name="DNP_top" color="12" fill="1" visible="yes" active="yes"/>
 <layer number="134" name="DNP_btm" color="12" fill="1" visible="no" active="yes"/>
 <layer number="144" name="Drill_legend" color="7" fill="1" visible="no" active="no"/>
@@
 <element name="R8" library="EEZ_Lib1" package="R_2512-4WIRE" value="GMR100HTBFIR022" x="28.4988" y="34.6583" smashed="yes" rot="R90">
 <attribute name="NAME" x="24.6634" y="34.1884" size="1.016" layer="25" ratio="10"/>
-<attribute name="VALUE" x="28.7909" y="30.8356" size="0.6096" layer="27" ratio="10" rot="R90"/>
+<attribute name="VALUE" x="28.8036" y="31.0134" size="0.6096" layer="27" ratio="10" rot="R90"/>
 </element>
 <element name="R26" library="rcl" package="R0805" value="330R" x="99.1616" y="14.8209" smashed="yes" rot="R90">
@@
 <element name="JP6" library="EEZ_Lib1" package="2MM-2" value="DS1025-01-1*2P8BV1-B" x="94.361" y="45.0469" smashed="yes">
 <attribute name="NAME" x="93.2688" y="47.0916" size="0.8128" layer="25" ratio="10"/>
-<attribute name="VALUE" x="94.8563" y="44.6786" size="0.4064" layer="27" ratio="10" rot="R90" align="center"/>
+<attribute name="VALUE" x="94.3483" y="45.1104" size="0.4064" layer="27" ratio="10" rot="R90" align="center"/>
 </element>
 <element name="IC6" library="EEZ_TI" package="DBV5" value="MCP6001T-I/OT" x="93.7006" y="33.8455" smashed="yes" rot="R90">
@@
 <attribute name="VALUE" x="69.977" y="47.6377" size="1.27" layer="27" ratio="10" rot="R180"/>
 </element>
-<element name="R30" library="rcl" package="R1206" value="33R" x="88.1761" y="41.8338" smashed="yes">
+<element name="R30" library="rcl" package="R1206" value="20R" x="88.1761" y="41.8338" smashed="yes">
 <attribute name="NAME" x="90.8685" y="41.529" size="0.8128" layer="25" ratio="10"/>
-<attribute name="VALUE" x="86.6521" y="41.3512" size="1.016" layer="27" ratio="10"/>
+<attribute name="VALUE" x="86.9569" y="41.275" size="1.016" layer="27" ratio="10"/>
 </element>
 <element name="R33" library="rcl" package="R0805" value="10K" x="96.7867" y="32.0929" smashed="yes" rot="R270">
@@
 <attribute name="OC_FARNELL" value="1713823" x="69.342" y="-46.6344" size="0.8128" layer="27" ratio="10" display="off"/>
 <attribute name="NAME" x="93.4339" y="39.5351" size="1.016" layer="25" ratio="10" rot="SR0"/>
-<attribute name="VALUE" x="92.5068" y="36.4236" size="0.4064" layer="27" ratio="10" rot="SR90"/>
+<attribute name="VALUE" x="90.6526" y="39.7256" size="0.4064" layer="27" ratio="10" rot="SR0"/>
 </element>
 <element name="Q4" library="EEZ_Lib1" package="SOT103P240X110-3N" value="BSS214NH6327XTSA1" x="89.0524" y="38.8874" smashed="yes">
@@
 <attribute name="OC_FARNELL" value="1713823" x="45.1485" y="-53.9242" size="0.8128" layer="27" ratio="10" display="off"/>
 <attribute name="NAME" x="88.5571" y="36.195" size="1.016" layer="25" ratio="10" rot="SR0"/>
-<attribute name="VALUE" x="90.3478" y="40.132" size="0.4064" layer="27" ratio="10" rot="SR180"/>
+<attribute name="VALUE" x="83.8835" y="37.6809" size="0.4064" layer="27" ratio="10" rot="SR0"/>
 </element>
 <element name="R36" library="rcl" package="R1206" value="100K" x="82.4357" y="40.6527" smashed="yes" rot="R180">
