File: EDA files/EEZ DIB AFE3 r1B4.brd (EAGLE design)
At the start: 129 x 68.5 mm, 149 parts, among them IC1 AMC3330QDWERQ1, IC11 ADS131E04IPAGR, IC12 TPS71725DCKR, IC13 TPS72325DBVR, IC2 ULN2803ADWR, IC3 AMC3301DWER, IC4 MCP6004T-I/ST, IC5 DG212BDY-T1-E3, IC6 MCP6001T-I/OT, IC7 DG212BDY-T1-E3, IC8 N.C., Q1 CPC3902ZTR, Q2 CPC3902ZTR, Q3 BSS214NH6327XTSA1, Q4 BSS214NH6327XTSA1, X1 691322310008, X2 DS1023-2*14S21, X3 DS1023-2*14S21

Commit message: Gerbers, BOM, schematics update
Parts:
- removed C47: 100n, rcl:C0603
- removed C48, C49: 1u, rcl:C0805
- removed C64: 10u, rcl:C1206
- removed F5: ZH32 (1.25A), EEZ_Lib1:ZH32
- removed IC13: TPS72325DBVR, EEZ_TI:DBV5
- removed JP9: JP2-CUT-0805, EEZ_Lib1:R_0805
- removed OK3: VOR1142B4, EEZ_DIB:DIL4-SMD
- removed Q3, Q4: BSS214NH6327XTSA1, EEZ_Lib1:SOT103P240X110-3N
- removed R38: 200K 0.1%, rcl:R1206
- removed R39: 100K 0.1%, rcl:R1206
- removed R51, R52: 10K, rcl:R0805
- removed R53, R54: 10R, rcl:R0805
- removed R65: N.C., rcl:R0805
- removed TVS1: PESD12VL1BA,115, EEZ_Lib1:SOD323-BIDIR
- added C29, C32: 100n, rcl:C0603
- added C30: 22u, rcl:C1206
- added C31: 10u, rcl:C1206
- added IC9: ADS131E04IPAGR, EEZ_TI:PAG64
- added JP7: JP3-CUT-0805-ROTATED, EEZ_Lib1:JP3-0805-CUT2
- C27: value 1u -> N.C.; device rcl:C0805 -> rcl:C1206
- C28: value 100n -> 1u; device rcl:C0603 -> rcl:C0805
- C33: value 22u -> 100n; device rcl:C1206 -> rcl:C0603
- C34: value 10u -> 1u; device rcl:C1206 -> rcl:C0805
- C35: value N.C. -> 1u; device rcl:C1206 -> rcl:C0805
- C46: value 100n -> 10u; device rcl:C0603 -> rcl:C1206
- F3: value SN005-60 -> ZH32 (1.25A); device EEZ_Lib1:C1206-HV -> EEZ_Lib1:ZH32
- IC11: value ADS131E04IPAGR -> TPS72325DBVR; device EEZ_TI:PAG64 -> EEZ_TI:DBV5
- IC6: value MCP6001T-I/OT -> DG212BDY-T1-E3; device EEZ_TI:DBV5 -> EEZ_DIB:SO16
- IC7: value DG212BDY-T1-E3 -> MCP6001T-I/OT; device EEZ_DIB:SO16 -> EEZ_TI:DBV5
- JP8: value JP3-CUT-0805-ROTATED -> JP2-CUT-0805; device EEZ_Lib1:JP3-0805-CUT2 -> EEZ_Lib1:R_0805
- Q1, Q2: value CPC3902ZTR -> BSS214NH6327XTSA1; device EEZ_Lib1:SOT230P700X180-4N -> EEZ_Lib1:SOT103P240X110-3N
- R13: value 10R -> 470R
- R14: value 470R -> 49K9; device rcl:R0805 -> rcl:R1206
- R15: value 33R 0.1% -> 49K9
- R16: value 470R -> 100K; device rcl:R0805 -> rcl:R1206
- R17, R18: value 49K9 -> 4M7 0.1%
- R19: value 100K -> 100K 0.1%
- R20, R21: value 4M7 0.1% -> 200K 0.1%
- R23: value 200K 0.1% -> 330R; device rcl:R1206 -> rcl:R0805
- R24: value 200K 0.1% -> 10K; device rcl:R1206 -> rcl:R0805
- R25: value 100K 0.1% -> 10K; device rcl:R1206 -> rcl:R0805
- R27: value 10K -> 33R; device rcl:R0805 -> rcl:R1206
- R28: value 10K -> 100K; device rcl:R0805 -> rcl:R1206
- R29: value 330R -> GMR100HTBFIR022; device rcl:R0805 -> EEZ_Lib1:R_2512-4WIRE
- R30: value 20R -> 10K; device rcl:R1206 -> rcl:R0805
- R31: value 100K -> 1K; device rcl:R1206 -> rcl:R0805
- R32: value GMR100HTBFIR022 -> GMR100HTBFA10L0
- R33: value 10K -> N.C.
- R34: value 1K -> 10K
- R35: value GMR100HTBFA10L0 -> 10K; device EEZ_Lib1:R_2512-4WIRE -> rcl:R0805
- R36: value 100K -> 10R; device rcl:R1206 -> rcl:R0805
- R37: value 200K 0.1% -> 10R; device rcl:R1206 -> rcl:R0805
- moved R37 53.0 mm to (119.7, 8.71), turned to 180 degrees
- moved R36 45.1 mm to (117.8, 12.7)
- moved R35 39.4 mm to (123.1, 37.7)
- moved C35 36.0 mm to (117.0, 6.29), turned to 180 degrees
- moved R23 34.0 mm to (99.2, 14.8), turned to 90 degrees
- moved R34 33.8 mm to (124.3, 16.3), turned to 270 degrees
- moved R24 33.7 mm to (101.1, 14.8), turned to 270 degrees
- moved R27 30.0 mm to (88.2, 41.8), turned to 0 degrees
- moved F3 29.5 mm to (65.2, 47.1), turned to 180 degrees
- moved R25 29.0 mm to (94.9, 27.0), turned to 270 degrees
- moved C46 25.9 mm to (110.5, 36.4), turned to 90 degrees
- moved C27 25.5 mm to (117.3, 42.3)
- moved R22 25.3 mm to (87.0, 23.2)
- moved R21 25.3 mm to (82.0, 23.2)
- moved R20 25.3 mm to (77.1, 23.2)
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- renumbered C54 to C36, C55 to C37, C56 to C38, C57 to C39, C58 to C40, C59 to C41, C60 to C42, C61 to C43, C62 to C44, C63 to C45, IC12 to IC10
Connections:
- removed net AIN_U4: ISEL1A_1.10, ISEL1A_1.3, JP2.2, R36.2, R37.2, TVS1.C2
- removed net CURR#3: IC5.11, Q2.2, Q2.4, R15.2
- removed net CURR_IN#3: OK2.3, Q1.2, Q1.4
- removed net ISEL#3: IC5.9, R14.2, X3.15
- removed net N$187: R37.1, R38.2
- removed net N$189: IC7.2, R38.1, R39.2
- removed net N$192: IC7.6, R36.1
- removed net N$58: OK3.3, R18.1
- removed net N$62: IC5.3, R22.1, R23.2
- removed net N$63 (its old number): R23.1, R24.2
- removed net N$66: OK2.1, R14.1
- removed net N$68: F3.2, Q1.1, Q2.3
- removed net N$69: Q1.3, Q2.1, R13.2
- removed net N$72: F3.1, R13.1
- removed net USEL1#4: IC7.8, X3.12
- removed net USEL5#4: IC7.1, X3.14
- new net AIN3/20: IC5.3, R19.1, R20.2
- new net N$18: OK2.4, R14.2
- new net N$61: R14.1, R15.2
- net !ADC_CS: now also IC9.39; no longer IC11.39
- net !ADC_DRDY: now also IC9.47; no longer IC11.47
- net !RESET: now also IC9.36; no longer IC11.36
- net +15V_ISO: now also IC6.13; no longer IC7.13
- net +2V5_ADC: now also IC9.19, IC9.21, IC9.22, IC9.54, IC9.56, IC9.59, R36.2; no longer IC11.19, IC11.21, IC11.22, IC11.54, IC11.56, IC11.59, R53.2
- net +2V5_ISO: now also C34.2, IC7.5, R23.1, R36.1; no longer C48.2, IC6.5, R26.1, R53.1
- net +3V3_ISO: now also IC9.48, IC9.50, JP7.NC, R34.2; no longer IC11.48, IC11.50, JP8.NC, R51.2
- net +5V_ISO: now also IC6.12; no longer IC7.12
- net -15V_ISO: now also IC6.4; no longer IC7.4
- net -2V5_ISO: now also C35.2, IC11.5, IC7.2, R26.2, R37.2; no longer C49.2, IC13.5, IC6.2, R29.2, R54.2
- net ADC_CLK: now also JP8.1; no longer JP9.1
- net ADC_MISO: now also IC9.43; no longer IC11.43
- net ADC_MOSI: now also IC9.34; no longer IC11.34
- net ADC_SCK: now also IC9.40; no longer IC11.40
- net ADC_START: now also IC9.38; no longer IC11.38
- net AIN3P: now also OK2.3; no longer JP4.2, OK2.4, R20.2
- net AIN4N: now also R28.2, R32.1; no longer R31.2, R35.1, TVS1.C1
- net AIN4P: now also F3.2; no longer F5.2
- net AIN4P_FUSED: now also F3.1; no longer F5.1
- net AVSS: now also C28.1, C29.2, C30.1, C31.2, C46.1, IC9.20, IC9.23, IC9.25, IC9.32, IC9.53, IC9.57, IC9.58, R33.2, R37.1; no longer C27.1, C28.2, C33.1, C34.2, C64.1, IC11.20, IC11.23, IC11.25, IC11.32, IC11.53, IC11.57, IC11.58, R54.1, R65.2
- net GND: now also C32.2, C33.2, C34.1, C35.1, IC11.1, IC6.5, IC9.31, IC9.33, IC9.41, IC9.49, IC9.51, JP7.NO, R16.1, R24.2, R25.1; no longer C47.2, C48.1, C49.1, C64.2, IC11.31, IC11.33, IC11.41, IC11.49, IC11.51, IC13.1, IC7.5, JP8.NO, OK3.2, R19.1, R27.2, R31.1
- net HI_CLAMP: now also R23.2, R24.1; no longer R26.2, R27.1
- net HI_CURR#1: now also R32.2; no longer R35.2
- net IN1N: now also IC9.15; no longer IC11.15
- net IN1P: now also IC9.16; no longer IC11.16
- net IN2N: now also IC9.13; no longer IC11.13
- net IN2P: now also IC9.14; no longer IC11.14
- net IN3N: now also IC9.11, R16.2, R22.1; no longer IC11.11, R15.1, R19.2, R25.1
- net IN3P: now also IC9.12, JP4.2; no longer IC11.12, IC5.10
- net IN4N: now also IC9.9, R32.1S; no longer IC11.9, R35.1S, R39.1
- net IN4P: now also IC6.11, IC6.15, IC9.10, JP2.2; no longer IC11.10, IC7.11, IC7.15, IC7.3, IC7.7
- net ISEL_LOW#4: now also IC6.16; no longer IC7.16
- net ISEL_MID#4: now also IC6.9, Q1.1, Q2.1; no longer IC7.9, Q3.1, Q4.1
- net LO_CLAMP: now also R25.2, R26.1; no longer R28.2, R29.1
- net N$1: now also IC9.52, R35.1; no longer IC11.52, R52.1
- net N$100: now also C27.2, R33.1; no longer C35.2, R65.1
- net N$14: now also JP7.COM, R35.2; no longer JP8.COM, R52.2
- net N$170: now also Q2.2, R27.1, R29.2; no longer Q4.2, R30.1, R32.2
- net N$173: now also R31.2; no longer R34.2
- net N$182: now also IC6.14, Q1.2, R27.2; no longer IC7.14, Q3.2, R33.2
- net N$183: now also IC7.1, IC7.4, R31.1; no longer IC6.1, IC6.4, R34.1
- net N$184: now also IC7.3, R30.1; no longer IC6.3, R33.1
- net N$19: now also R29.1, R29.1S, R32.2S; no longer R32.1, R32.1S, R35.2S
- net N$27: now also IC6.10, R29.2S; no longer IC7.10, R32.2S
- net N$3: now also C32.1; no longer C46.1
- net N$56: now also R21.1, R22.2; no longer R24.1, R25.2
- net N$57: now also R15.1; no longer OK3.4
- net N$64: now also R18.1, R19.2; no longer R21.1, R22.2
- net N$67: now also OK2.1, R13.2; no longer OK3.1, R16.2
- net N$81: now also Q1.3, Q2.3; no longer Q3.3, Q4.3
- net N$9: now also C33.1, IC11.2, IC11.3; no longer C47.1, IC13.2, IC13.3
- net N$92: now also C30.2, IC9.28; no longer C33.2, IC11.28
- net N$93: now also C28.2, IC9.30; no longer C27.2, IC11.30
- net N$94: now also IC9.55; no longer IC11.55
- net N$95: now also IC9.26; no longer IC11.26
- net N$96: now also IC9.37, JP8.2; no longer IC11.37, JP9.2
- net N$98: now also IC9.35, R34.1; no longer IC11.35, R51.1
- net USEL1#3: now also R13.1; no longer R16.1
- net VREFP: now also C27.1, C29.1, C31.1, IC9.24; no longer C28.1, C34.1, C35.1, IC11.24
Routing:
- net ISEL#3: track 77.2 -> 0.00 mm, vias 5 -> 0
- net USEL1#4: track 44.0 -> 0.00 mm, vias 2 -> 0
- net USEL5#4: track 40.8 -> 0.00 mm, vias 2 -> 0
- net N$62: track 31.1 -> 0.00 mm, vias 2 -> 0
- net AIN3P: track 39.0 -> 8.83 mm, vias 3 -> 0
- net IN3P: track 46.3 -> 72.5 mm
- net AIN_U4: track 24.2 -> 0.00 mm
- net N$189: track 23.7 -> 0.00 mm, vias 2 -> 0
- net AIN3/20: track 0.00 -> 19.3 mm, vias 0 -> 2
- net N$192: track 15.1 -> 0.00 mm, vias 2 -> 0
- net CURR#3: track 13.8 -> 0.00 mm
- net IN3N: track 131.4 -> 144.2 mm
- net N$56: track 28.8 -> 16.8 mm
- net +3V3_ISO: track 79.8 -> 91.3 mm
- net N$13: track 44.3 -> 54.9 mm, vias 2 -> 1
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- removed copper zone on layer 1, net CURR#3
- removed copper zone on layer 1, net CURR_IN#3
Other:
- board text added: "EEZ DIB AFE3 (08/2021 r1B4)"
- board text removed: "EEZ DIB AFE3 (05/2021 r1B3)"
