File: EDA files/EEZ DIB AFE3 r1B4.sch (EAGLE design)
At the start: 148 parts, among them IC1 AMC3330QDWERQ1, IC11 ADS131E04IPAGR, IC12 TPS71725DCKR, IC13 TPS72325DBVR, IC2 ULN2803ADWR, IC3 AMC3301DWER, IC4 MCP6004T-I/ST, IC5 DG212BDY-T1-E3, IC6 MCP6001T-I/OT, IC7 DG212BDY-T1-E3, IC8 N.C., Q1 CPC3902ZTR, Q2 CPC3902ZTR, Q3 BSS214NH6327XTSA1, Q4 BSS214NH6327XTSA1, X1 691322310008, X2 DS1023-2*14S21, X3 DS1023-2*14S21

Commit message: Gerbers, BOM, schematics update
Parts:
- removed C47: 100n, rcl:C-EUC0603
- removed C48, C49: 1u, rcl:C-EUC0805
- removed C64: 10u, rcl:C-EUC1206
- removed F5: ZH32 (1.25A), EEZ_Lib1:ZH32
- removed IC13: TPS72325DBVR, EEZ_TI:TPS72325DBVR
- removed JP9: JP2-CUT-0805, EEZ_Lib1:JP2-CUT-0805
- removed OK3: VOR1142B4, EEZ_DIB:VOR1142B4
- removed Q3, Q4: BSS214NH6327XTSA1, EEZ_Lib1:2N7002
- removed R38: 200K 0.1%, rcl:R-EU_R1206
- removed R39: 100K 0.1%, rcl:R-EU_R1206
- removed R51, R52: 10K, rcl:R-EU_R0805
- removed R53, R54: 10R, rcl:R-EU_R0805
- removed R65: N.C., rcl:R-EU_R0805
- removed TVS1: PESD12VL1BA,115, EEZ_Lib1:PESDXL1BA
- added C29, C32: 100n, rcl:C-EUC0603
- added C30: 22u, rcl:C-EUC1206
- added C31: 10u, rcl:C-EUC1206
- added IC9: ADS131E04IPAGR, EEZ_TI:ADS131E0XIPAG
- added JP7: JP3-CUT-0805-ROTATED, EEZ_Lib1:JP3-CUT-0805-ROTATED
- C27: value 1u -> N.C.; device rcl:C-EUC0805 -> rcl:C-EUC1206
- C28: value 100n -> 1u; device rcl:C-EUC0603 -> rcl:C-EUC0805
- C33: value 22u -> 100n; device rcl:C-EUC1206 -> rcl:C-EUC0603
- C34: value 10u -> 1u; device rcl:C-EUC1206 -> rcl:C-EUC0805
- C35: value N.C. -> 1u; device rcl:C-EUC1206 -> rcl:C-EUC0805
- C46: value 100n -> 10u; device rcl:C-EUC0603 -> rcl:C-EUC1206
- F3: value SN005-60 -> ZH32 (1.25A); device EEZ_Lib1:FUSE_RESETTABLE2 -> EEZ_Lib1:ZH32
- IC11: value ADS131E04IPAGR -> TPS72325DBVR; device EEZ_TI:ADS131E0XIPAG -> EEZ_TI:TPS72325DBVR
- IC6: value MCP6001T-I/OT -> DG212BDY-T1-E3; device EEZ_TI:OPA376AIDBVR -> EEZ_DIB:DG212BDY-T1-E3
- IC7: value DG212BDY-T1-E3 -> MCP6001T-I/OT; device EEZ_DIB:DG212BDY-T1-E3 -> EEZ_TI:OPA376AIDBVR
- JP8: value JP3-CUT-0805-ROTATED -> JP2-CUT-0805; device EEZ_Lib1:JP3-CUT-0805-ROTATED -> EEZ_Lib1:JP2-CUT-0805
- Q1: value CPC3902ZTR -> BSS214NH6327XTSA1; device EEZ_Lib1:BSP129SOT-223 -> EEZ_Lib1:2N7002; MPN (none) -> 2N7002-7-F; OC_FARNELL (none) -> 1713823; OC_NEWARK (none) -> 25R5679; PACKAGE (none) -> SOT-23-3; SUPPLIER (none) -> DIODES INC.
- Q2: value CPC3902ZTR -> BSS214NH6327XTSA1; device EEZ_Lib1:BSP129SOT-223 -> EEZ_Lib1:2N7002
- R13: value 10R -> 470R
- R14: value 470R -> 49K9; device rcl:R-EU_R0805 -> rcl:R-EU_R1206
- R15: value 33R 0.1% -> 49K9
- R16: value 470R -> 100K; device rcl:R-EU_R0805 -> rcl:R-EU_R1206
- R17, R18: value 49K9 -> 4M7 0.1%
- R19: value 100K -> 100K 0.1%
- R20, R21: value 4M7 0.1% -> 200K 0.1%
- R23: value 200K 0.1% -> 330R; device rcl:R-EU_R1206 -> rcl:R-EU_R0805
- R24: value 200K 0.1% -> 10K; device rcl:R-EU_R1206 -> rcl:R-EU_R0805
- R25: value 100K 0.1% -> 10K; device rcl:R-EU_R1206 -> rcl:R-EU_R0805
- R27: value 10K -> 33R; device rcl:R-EU_R0805 -> rcl:R-EU_R1206
- R28: value 10K -> 100K; device rcl:R-EU_R0805 -> rcl:R-EU_R1206
- R29: value 330R -> GMR100HTBFIR022; device rcl:R-EU_R0805 -> EEZ_Lib1:R-EU_4WIRE2512
- R30: value 20R -> 10K; device rcl:R-EU_R1206 -> rcl:R-EU_R0805
- R31: value 100K -> 1K; device rcl:R-EU_R1206 -> rcl:R-EU_R0805
- R32: value GMR100HTBFIR022 -> GMR100HTBFA10L0
- R33: value 10K -> N.C.
- R34: value 1K -> 10K
- R35: value GMR100HTBFA10L0 -> 10K; device EEZ_Lib1:R-EU_4WIRE2512 -> rcl:R-EU_R0805
- R36: value 100K -> 10R; device rcl:R-EU_R1206 -> rcl:R-EU_R0805
- R37: value 200K 0.1% -> 10R; device rcl:R-EU_R1206 -> rcl:R-EU_R0805
- renumbered C54 to C36, C55 to C37, C56 to C38, C57 to C39, C58 to C40, C59 to C41, C60 to C42, C61 to C43, C62 to C44, C63 to C45, IC12 to IC10
Connections:
- removed net AIN_U4: ISEL1A_1B.NC, ISEL1A_1C.NC, JP2.2, R36.2, R37.2, TVS1.2
- removed net CURR#3: IC5C.S, Q2.D, R15.2
- removed net CURR_IN#3: OK2.S2, Q1.D
- removed net ISEL#3: IC5C.IN, R14.2, X3-15.1
- removed net N$187: R37.1, R38.2
- removed net N$189: IC7A.D, R38.1, R39.2
- removed net N$192: IC7D.S, R36.1
- removed net N$58: OK3.S2, R18.1
- removed net N$62: IC5A.S, R22.1, R23.2
- removed net N$63 (its old number): R23.1, R24.2
- removed net N$66: OK2.A, R14.1
- removed net N$68: F3.P$2, Q1.G, Q2.S
- removed net N$69: Q1.S, Q2.G, R13.2
- removed net N$72: F3.P$1, R13.1
- removed net USEL1#4: IC7D.IN, X3-12.1
- removed net USEL5#4: IC7A.IN, X3-14.1
- new net AIN3/20: IC5A.S, R19.1, R20.2
- new net N$18: OK2.S1, R14.2
- new net N$61: R14.1, R15.2
- net !ADC_CS: now also IC9.!CS; no longer IC11.!CS
- net !ADC_DRDY: now also IC9.!DRDY; no longer IC11.!DRDY
- net !RESET: now also IC9.!RESET; no longer IC11.!RESET
- net +15V_ISO: now also IC6P.V+; no longer IC7P.V+
- net +2V5_ADC: now also IC9.AVDD, IC9.AVDD1, IC9.AVDD_2, IC9.AVDD_3, IC9.AVDD_4, IC9.AVDD_5, R36.2; no longer IC11.AVDD, IC11.AVDD1, IC11.AVDD_2, IC11.AVDD_3, IC11.AVDD_4, IC11.AVDD_5, R53.2
- net +2V5_ISO: now also C34.2, IC7P.V+, R23.1, R36.1; no longer C48.2, IC6P.V+, R26.1, R53.1
- net +3V3_ISO: now also IC9.DVDD, IC9.DVDD_2, JP7.NC, R34.2; no longer IC11.DVDD, IC11.DVDD_2, JP8.NC, R51.2
- net +5V_ISO: now also IC6P.VL; no longer IC7P.VL
- net -15V_ISO: now also IC6P.V-; no longer IC7P.V-
- net -2V5_ISO: now also C35.2, IC11.OUT, IC7P.V-, R26.2, R37.2; no longer C49.2, IC13.OUT, IC6P.V-, R29.2, R54.2
- net ADC_CLK: now also JP8.1; no longer JP9.1
- net ADC_MISO: now also IC9.DOUT; no longer IC11.DOUT
- net ADC_MOSI: now also IC9.DIN; no longer IC11.DIN
- net ADC_SCK: now also IC9.SCLK; no longer IC11.SCLK
- net ADC_START: now also IC9.START; no longer IC11.START
- net AIN3P: now also OK2.S2; no longer JP4.2, OK2.S1, R20.2
- net AIN4N: now also R28.2, R32.1; no longer R31.2, R35.1, TVS1.1
- net AIN4P: now also F3.2; no longer F5.2
- net AIN4P_FUSED: now also F3.1; no longer F5.1
- net AVSS: now also C28.1, C29.2, C30.1, C31.2, C46.1, IC9.AVSS, IC9.AVSS1, IC9.AVSS_2, IC9.AVSS_3, IC9.AVSS_4, IC9.AVSS_5, IC9.VREFN, R33.2, R37.1; no longer C27.1, C28.2, C33.1, C34.2, C64.1, IC11.AVSS, IC11.AVSS1, IC11.AVSS_2, IC11.AVSS_3, IC11.AVSS_4, IC11.AVSS_5, IC11.VREFN, R54.1, R65.2
- net GND: now also C32.2, C33.2, C34.1, C35.1, IC11.GND, IC6P.GND, IC9.DAISY_IN, IC9.DGND, IC9.DGND_2, IC9.DGND_3, IC9.RESV1, JP7.NO, R16.1, R24.2, R25.1; no longer C47.2, C48.1, C49.1, C64.2, IC11.DAISY_IN, IC11.DGND, IC11.DGND_2, IC11.DGND_3, IC11.RESV1, IC13.GND, IC7P.GND, JP8.NO, OK3.C, R19.1, R27.2, R31.1
- net HI_CLAMP: now also R23.2, R24.1; no longer R26.2, R27.1
- net HI_CURR#1: now also R32.2; no longer R35.2
- net IN1N: now also IC9.IN1N; no longer IC11.IN1N
- net IN1P: now also IC9.IN1P; no longer IC11.IN1P
- net IN2N: now also IC9.IN2N; no longer IC11.IN2N
- net IN2P: now also IC9.IN2P; no longer IC11.IN2P
- net IN3N: now also IC9.IN3N, R16.2, R22.1; no longer IC11.IN3N, R15.1, R19.2, R25.1
- net IN3P: now also IC9.IN3P, JP4.2; no longer IC11.IN3P, IC5C.D
- net IN4N: now also IC9.IN4N, R32.1S; no longer IC11.IN4N, R35.1S, R39.1
- net IN4P: now also IC6B.D, IC6C.S, IC9.IN4P, JP2.2; no longer IC11.IN4P, IC7A.S, IC7B.D, IC7C.S, IC7D.D
- net ISEL_LOW#4: now also IC6B.IN; no longer IC7B.IN
- net ISEL_MID#4: now also IC6C.IN, Q1.G, Q2.G; no longer IC7C.IN, Q3.G, Q4.G
- net LO_CLAMP: now also R25.2, R26.1; no longer R28.2, R29.1
- net N$1: now also IC9.CLKSEL, R35.1; no longer IC11.CLKSEL, R52.1
- net N$100: now also C27.2, R33.1; no longer C35.2, R65.1
- net N$14: now also JP7.COM, R35.2; no longer JP8.COM, R52.2
- net N$170: now also Q2.S, R27.1, R29.2; no longer Q4.S, R30.1, R32.2
- net N$173: now also R31.2; no longer R34.2
- net N$182: now also IC6B.S, Q1.S, R27.2; no longer IC7B.S, Q3.S, R33.2
- net N$183: now also IC7A.-IN, IC7A.OUT, R31.1; no longer IC6A.-IN, IC6A.OUT, R34.1
- net N$184: now also IC7A.+IN, R30.1; no longer IC6A.+IN, R33.1
- net N$19: now also R29.1, R29.1S, R32.2S; no longer R32.1, R32.1S, R35.2S
- net N$27: now also IC6C.D, R29.2S; no longer IC7C.D, R32.2S
- net N$3: now also C32.1; no longer C46.1
- net N$56: now also R21.1, R22.2; no longer R24.1, R25.2
- net N$57: now also R15.1; no longer OK3.S1
- net N$64: now also R18.1, R19.2; no longer R21.1, R22.2
- net N$67: now also OK2.A, R13.2; no longer OK3.A, R16.2
- net N$81: now also Q1.D, Q2.D; no longer Q3.D, Q4.D
- net N$9: now also C33.1, IC11.EN, IC11.IN; no longer C47.1, IC13.EN, IC13.IN
- net N$92: now also C30.2, IC9.VCAP1; no longer C33.2, IC11.VCAP1
- net N$93: now also C28.2, IC9.VCAP2; no longer C27.2, IC11.VCAP2
- net N$94: now also IC9.VCAP3; no longer IC11.VCAP3
- net N$95: now also IC9.VCAP4; no longer IC11.VCAP4
- net N$96: now also IC9.CLK, JP8.2; no longer IC11.CLK, JP9.2
- net N$98: now also IC9.!PWDN, R34.1; no longer IC11.!PWDN, R51.1
- net USEL1#3: now also R13.1; no longer R16.1
- net VREFP: now also C27.1, C29.1, C31.1, IC9.VREFP; no longer C28.1, C34.1, C35.1, IC11.VREFP
Other:
- note added: "Current mode: ±48 mA (gain x1), ±500 mA (gain x2), ±10 A (gain x12)"
- note added: "Voltage mode: ±2.4 V, ±48 V, ±240 V"
- note added: "Voltage ranges: ±50 V, ±480 V"
- note removed: "Dovesti na ADIB AIN1 i AIN2 !!!"
- note removed: "Voltage mode: ±2.4 V, ±12 V Current mode: ±48 mA (gain x1), ±1.2 A (gain x2), ±10 A (gain x12)"
- note removed: "Voltage mode: ±2.4 V, ±48 V, ±240 V Current mode: ±48 mA (gain x1)"
- note removed: "Voltage ranges: ±55 V, ±480 V"
- note removed: "÷5"
